File: PCB/Macropad.kicad_pcb (KiCad board)
At the start: 2 copper layers, 84.2 x 91.2 mm, 26 parts, among them SW1 RotaryEncoder_Switch, SW2 SW_Push, SW3 SW_Push, SW4 SW_Push, SW5 SW_Push, SW6 SW_Push, SW7 SW_Push, SW8 SW_Push, SW9 SW_Push, U1 XIAO-RP2040-DIP

Commit message: Add files via upload
Parts:
- D1, D2, D3, D4, D5, D6, D7, D8, D9: footprint Diode_SMD:D_SOD-523 -> Diode_THT:D_DO-35_SOD27_P7.62mm_Horizontal
- moved D4 5.75 mm to (92.8, 90.8)
- moved D1 4.79 mm to (74.3, 90.5)
- moved D3 4.41 mm to (109.7, 90.2)
- moved D5 4.14 mm to (73.7, 127.3)
- moved D6 3.93 mm to (111.5, 127.7)
- moved D8 3.91 mm to (74.3, 108.0)
- moved D9 3.71 mm to (92.8, 109.2)
- moved D7 3.13 mm to (92.8, 127.0)
- moved D2 2.99 mm to (110.8, 109.2)
Routing:
- net R2: track 169.9 -> 155.5 mm
- net R1: track 139.9 -> 127.8 mm
- net Net-(D8-A): track 31.9 -> 36.8 mm
- net R3: track 149.5 -> 153.5 mm
- net Net-(D3-A): track 50.1 -> 54.2 mm
- net Net-(D9-A): track 6.45 -> 10.4 mm
- net Net-(D2-A): track 61.5 -> 57.8 mm
- net Net-(D6-A): track 80.0 -> 76.9 mm

Commit message: Add files via upload
Connections:
- SW3 pad 1: Net-(SW3-Pad1) -> C1
- SW5 pad 1: Net-(SW3-Pad1) -> C1
Routing:
- net C1: track 34.6 -> 96.4 mm, vias 1 -> 3
- net Net-(SW3-Pad1): track 19.1 -> 0.00 mm
Changed lines of the file:
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@@
 	(net 26 "Rotary_B")
 	(net 27 "C2")
-	(net 28 "Net-(SW3-Pad1)")
-	(net 29 "C3")
-	(net 30 "unconnected-(U1-3V3-Pad12)")
+	(net 28 "C3")
+	(net 29 "unconnected-(U1-3V3-Pad12)")
 	(footprint "Button_Switch_Keyboard:SW_Cherry_MX_1.00u_PCB"
 		(layer "F.Cu")
@@
 			(layers "*.Cu" "*.Mask")
 			(remove_unused_layers no)
-			(net 29 "C3")
+			(net 28 "C3")
 			(pinfunction "1")
 			(pintype "passive")
@@
 			(layers "*.Cu" "*.Mask")
 			(remove_unused_layers no)
-			(net 29 "C3")
+			(net 28 "C3")
 			(pinfunction "GPIO1/RX")
 			(pintype "passive")
@@
 			(layers "F.Cu" "F.Mask" "F.Paste")
 			(roundrect_rratio 0.25)
-			(net 29 "C3")
+			(net 28 "C3")
 			(pinfunction "GPIO1/RX")
 			(pintype "passive")
@@
 			(layers "*.Cu" "*.Mask")
 			(remove_unused_layers no)
-			(net 30 "unconnected-(U1-3V3-Pad12)")
+			(net 29 "unconnected-(U1-3V3-Pad12)")
 			(pinfunction "3V3")
 			(pintype "passive")
@@
 			(layers "F.Cu" "F.Mask" "F.Paste")
 			(roundrect_rratio 0.25)
-			(net 30 "unconnected-(U1-3V3-Pad12)")
+			(net 29 "unconnected-(U1-3V3-Pad12)")
 			(pinfunction "3V3")
 			(pintype "passive")
@@
 			(layers "*.Cu" "*.Mask")
 			(remove_unused_layers no)
-			(net 29 "C3")
+			(net 28 "C3")
 			(pinfunction "1")
 			(pintype "passive")
@@
 			(layers "*.Cu" "*.Mask")
 			(remove_unused_layers no)
-			(net 28 "Net-(SW3-Pad1)")
+			(net 24 "C1")
 			(pinfunction "1")
 			(pintype "passive")
@@
 			(layers "*.Cu" "*.Mask")
 			(remove_unused_layers no)
-			(net 28 "Net-(SW3-Pad1)")
+			(net 24 "C1")
 			(pinfunction "1")
 			(pintype "passive")
@@
 			(layers "*.Cu" "*.Mask")
 			(remove_unused_layers no)
-			(net 29 "C3")
+			(net 28 "C3")
 			(pinfunction "1")
 			(pintype "passive")
@@
 	)
 	(segment
+		(start 71.89 111.27)
+		(end 71.79 111.17)
+		(width 0.2)
+		(layer "F.Cu")
+		(net 24)
+	)
+	(segment
 		(start 71.555 61.595)
 		(end 66.675 61.595)
@@
 	)
 	(segment
+		(start 71.79 111.17)
+		(end 71.79 96.26)
+		(width 0.2)
+		(layer "F.Cu")
+		(net 24)
+	)
+	(segment
+		(start 84.72472 99.695)
+		(end 75.05 109.36972)
+		(width 0.2)
+		(layer "F.Cu")
+		(net 24)
+	)
+	(segment
+		(start 85.56625 99.695)
+		(end 84.72472 99.695)
+		(width 0.2)
+		(layer "F.Cu")
+		(net 24)
+	)
+	(segment
+		(start 75.05 109.36972)
+		(end 75.05 111.27)
+		(width 0.2)
+		(layer "F.Cu")
+		(net 24)
+	)
+	(segment
+		(start 71.54375 93.16375)
+		(end 71.54375 88.225)
+		(width 0.2)
+		(layer "F.Cu")
+		(net 24)
+	)
+	(segment
+		(start 71.79 96.26)
+		(end 71.63 96.1)
+		(width 0.2)
+		(layer "F.Cu")
+		(net 24)
+	)
+	(segment
 		(start 71.85 61.75)
 		(end 71.71 61.75)
@@
 	)
 	(segment
+		(start 75.05 111.27)
+		(end 71.89 111.27)
+		(width 0.2)
+		(layer "F.Cu")
+		(net 24)
+	)
+	(segment
+		(start 85.56625 118.745)
+		(end 85.56625 99.695)
+		(width 0.2)
+		(layer "F.Cu")
+		(net 24)
+	)
+	(segment
 		(start 68.23 73.16)
 		(end 71.85 69.54)
@@
 		(net 24)
 	)
+	(segment
+		(start 71.59 93.21)
+		(end 71.54375 93.16375)
+		(width 0.2)
+		(layer "F.Cu")
+		(net 24)
+	)
+	(via
+		(at 71.59 93.21)
+		(size 0.6)
+		(drill 0.3)
+		(layers "F.Cu" "B.Cu")
+		(net 24)
+	)
+	(via
+		(at 71.63 96.1)
+		(size 0.6)
+		(drill 0.3)
+		(layers "F.Cu" "B.Cu")
+		(net 24)
+	)
 	(via
 		(at 68.23 73.16)
@@
 	)
 	(segment
+		(start 71.63 96.1)
+		(end 71.63 93.25)
+		(width 0.2)
+		(layer "B.Cu")
+		(net 24)
+	)
+	(segment
 		(start 71.54375 88.225)
 		(end 68.23 84.91125)
@@
 	)
 	(segment
+		(start 71.63 93.25)
+		(end 71.59 93.21)
+		(width 0.2)
+		(layer "B.Cu")
+		(net 24)
+	)
+	(segment
 		(start 49.98 73.3)
 		(end 50.955 72.325)
@@
 	)
 	(segment
-		(start 85.56625 118.745)
-		(end 85.56625 99.695)
-		(width 0.2)
-		(layer "F.Cu")
-		(net 28)
-	)
-	(segment
 		(start 104.61625 118.745)
 		(end 104.61625 99.695)
 		(width 0.2)
 		(layer "F.Cu")
-		(net 29)
+		(net 28)
 	)
 	(segment
@@
 		(width 0.2)
 		(layer "F.Cu")
-		(net 29)
+		(net 28)
 	)
 	(segment
@@
 		(width 0.2)
 		(layer "F.Cu")
-		(net 29)
+		(net 28)
 	)
 	(segment
@@
 		(width 0.2)
 		(layer "F.Cu")
-		(net 29)
+		(net 28)
 	)
 	(segment
@@
 		(width 0.2)
 		(layer "F.Cu")
-		(net 29)
+		(net 28)
 	)
 	(segment
@@
 		(width 0.2)
 		(layer "F.Cu")
-		(net 29)
+		(net 28)
 	)
 	(segment
@@
 		(width 0.2)
 		(layer "F.Cu")
-		(net 29)
+		(net 28)
 	)
 	(segment
@@
 		(width 0.2)
 		(layer "F.Cu")
-		(net 29)
+		(net 28)
 	)
 	(segment
@@
 		(width 0.2)
 		(layer "F.Cu")
-		(net 29)
+		(net 28)
 	)
 	(via
@@
 		(drill 0.3)
 		(layers "F.Cu" "B.Cu")
-		(net 29)
+		(net 28)
 	)
 	(via
@@
 		(drill 0.3)
 		(layers "F.Cu" "B.Cu")
-		(net 29)
+		(net 28)
 	)
 	(via
@@
 		(drill 0.3)
 		(layers "F.Cu" "B.Cu")
-		(net 29)
+		(net 28)
 	)
 	(segment
@@
 		(width 0.2)
 		(layer "B.Cu")
-		(net 29)
+		(net 28)
 	)
 	(segment
@@
 		(width 0.2)
 		(layer "B.Cu")
-		(net 29)
+		(net 28)
 	)
 	(segment
@@
 		(width 0.2)
 		(layer "B.Cu")
-		(net 29)
+		(net 28)
 	)
 	(segment
@@
 		(width 0.2)
 		(layer "B.Cu")
-		(net 29)
+		(net 28)
 	)
 	(segment
@@
 		(width 0.2)
 		(layer "B.Cu")
-		(net 29)
+		(net 28)
 	)
 	(segment
@@
 		(width 0.2)
 		(layer "B.Cu")
-		(net 29)
+		(net 28)
 	)
 	(segment
@@
 		(width 0.2)
 		(layer "B.Cu")
-		(net 29)
+		(net 28)
 	)
 	(segment
@@
 		(width 0.2)
 		(layer "B.Cu")
-		(net 29)
+		(net 28)
 	)
 	(embedded_fonts no)
